File: data/paste-flow-calibration-board/paste-flow-calibration-board.cricles_and_rectangles.kicad_pcb (KiCad board)
At the start: 2 copper layers, 47.5 x 20 mm, 91 parts

Commit message: feature(pasting): add paste dataset collection
Parts:
- renumbered PURGE1 to PURGE
Changed lines of the file:
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@@
 		(layer "F.Cu")
 		(at 1.25 1.25)
-		(property "Reference" "PURGE1"
+		(property "Reference" "PURGE"
 			(at 0 0 0)
 			(layer "F.SilkS")
